Commit message: add gazebo interface

File: urdf/hephaestus_calibration.urdf (robot description, URDF)
Before this commit: robot hephaestus_calbration, 7 links, 6 joints
Joints:
- joint joint1: limit lower=-3.141592653589793116 upper=3.141592653589793116 effort=1 velocity=20 -> lower=-3.141592653589793116 upper=3.141592653589793116 effort=20 velocity=20
- joint joint2: limit lower=-3.141592653589793116 upper=3.141592653589793116 effort=1 velocity=20 -> lower=-3.141592653589793116 upper=3.141592653589793116 effort=20 velocity=20
- joint joint3: limit lower=-3.141592653589793116 upper=3.141592653589793116 effort=1 velocity=20 -> lower=-3.141592653589793116 upper=3.141592653589793116 effort=20 velocity=20
- joint joint4: limit lower=-3.141592653589793116 upper=3.141592653589793116 effort=1 velocity=20 -> lower=-3.141592653589793116 upper=3.141592653589793116 effort=20 velocity=20
- joint joint5: limit lower=-3.141592653589793116 upper=3.141592653589793116 effort=1 velocity=20 -> lower=-3.141592653589793116 upper=3.141592653589793116 effort=20 velocity=20
- joint joint6: limit lower=-3.141592653589793116 upper=3.141592653589793116 effort=1 velocity=20 -> lower=-3.141592653589793116 upper=3.141592653589793116 effort=20 velocity=20
