Commit message: update urdf

File: urdf/hephaestus_description.urdf (robot description, URDF)
Before this commit: robot hephaestus_description, 7 links, 6 joints
Links:
- link gripper: mass 0.86773294449729154731 -> 0.89972887456439920584
- link link1: mass 0.037828410371921306066 -> 0.037828410371921313005; geometry collision mesh filename=package://hephaestus_description/meshes/base_link.stl; visual mesh filename=package://hephaestus_description/meshes/base_link.stl
- link link4: mass 0.86501392429453016764 -> 0.86501392429453005661
- link link5: mass 0.34991611054164151184 -> 0.34991611054164145633
- link link6: mass 0.34991611054164145633 -> 0.34991611054164140082
Joints:
- joint j3: axis 0 0 -1 -> 0 0 1
- joint j4: axis 0 0 -1 -> 0 0 1
- joint j5: axis 0 0 -1 -> 0 0 1
- joint j6: axis 0 0 -1 -> 0 0 1

Commit message: fixed direction of joints

File: urdf/hephaestus_description.urdf (robot description, URDF)
Before this commit: robot hephaestus_description, 7 links, 6 joints
Joints:
- joint j3: axis 0 0 1 -> 0 0 -1
- joint j4: axis 0 0 1 -> 0 0 -1
- joint j5: axis 0 0 1 -> 0 0 -1
- joint j6: axis 0 0 1 -> 0 0 -1

Commit message: update urdf

File: urdf/hephaestus_description.urdf (robot description, URDF)
Before this commit: robot hephaestus_description, 7 links, 6 joints
Links:
- link gripper: mass 0.89972887456439920584 -> 0.9115946721229465366; geometry collision mesh filename=package://hephaestus_description/meshes/4005_convertor.stl; collision mesh filename=package://hephaestus_description/meshes/4036_out_type_b.stl
- link link2: mass 1.0724812080404333425 -> 1.130266391889907629; geometry collision mesh filename=package://hephaestus_description/meshes/base.stl; collision mesh filename=package://hephaestus_description/meshes/flange.stl
- link link3: mass 2.4748694772611363746 -> 2.5487438908796358206; geometry collision mesh filename=package://hephaestus_description/meshes/aluminum_tube_11_32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; collision mesh filename=package://hephaestus_description/meshes/base.stl
- link link4: mass 0.86501392429453005661 -> 0.92830831261165880353; geometry collision mesh filename=package://hephaestus_description/meshes/aluminum_tube_11_32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; collision mesh filename=package://hephaestus_description/meshes/j3_converter_asm_1.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
- link link5: mass 0.34991611054164145633 -> 0.3646947997611872383; geometry collision mesh filename=package://hephaestus_description/meshes/4036_output_type_a.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; collision mesh filename=package://hephaestus_description/meshes/m3_6mm.stl
- link link6: mass 0.34991611054164140082 -> 0.36469479976118712727; geometry collision mesh filename=package://hephaestus_description/meshes/4036_output_type_a.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; collision mesh filename=package://hephaestus_description/meshes/m3_6mm.stl
Joints:
- joint j1: origin xyz=2.9298209278990825415e-31 -3.3306690738842268941e-19 0.0030000000000000004961 rpy=3.141592653589793116 2.2956344170608865771e-16 -1.570796326794896558 -> xyz=1.2094840050751841157e-30 -3.330669073883665004e-19 0.0030000000000000000625 rpy=-3.1415926535897922278 -2.0432878948499990369e-16 1.5707963267949001107
- joint j2: origin xyz=1.6386936912579358773e-15 -0.050000000000000113798 -0.061000000000003176681 rpy=-1.570796326794896558 2.8249375483975358926e-17 3.0864200084579932425e-14 -> xyz=6.5317576732167981012e-18 -0.049999999999999746036 -0.061000000000001497469 rpy=-1.5707963267948974462 1.1149798816950092785e-13 2.7183456743031896713e-16
- joint j3: origin xyz=4.0692392257585837815e-17 0.27900000000000046985 8.8817841970012523234e-16 rpy=-3.141592653589793116 1.956768080901109495e-15 -3.1415926535897926719 -> xyz=4.2971980656064264533e-14 0.27900000000004948619 6.3837823915946501074e-15 rpy=-3.1415926535896732119 -2.2411157873958029012e-15 3.1415926535896590011
- joint j4: origin xyz=-1.2582286762934820898e-16 0.27900000000000008127 -0.014500000000000047573 rpy=3.141592653589793116 -6.9410315361038256731e-16 -1.5707963267948961139 -> xyz=-8.3315527688767367743e-15 0.27900000000001856648 -0.014500000000024985958 rpy=-3.1415926535897913396 -1.0262745653896959069e-13 -1.5707963267948636954
- joint j5: origin xyz=-0.027499999999998525624 1.3193934789373790605e-16 -0.040500000000001007416 rpy=3.141592653589788231 -1.5707963267948452657 0 -> xyz=-0.027499999999995528022 8.9672221510033413429e-16 -0.040500000000003207046 rpy=3.1415926535897913396 -1.5707963267948412689 0
- joint j6: origin xyz=-1.3877787807814456755e-17 0.027499999999999961975 -0.040500000000000091482 rpy=1.5707963267948972241 1.5707963267948961139 0 -> xyz=-4.1633363423443370266e-17 0.027499999999999531763 -0.040499999999995317523 rpy=1.5707963267949276442 1.5707963267948825692 0

Commit message: modified link1's inertial for KDL

File: urdf/hephaestus_description.urdf (robot description, URDF)
Before this commit: robot hephaestus_description, 7 links, 6 joints
Links:
- added link link1_inertial, mass 0.037828410371921313005
- link link1: mass 0.037828410371921313005 -> None
Joints:
- added joint link1_inertial_joint: type fixed, parent link1, child link1_inertial, origin xyz=0 0 0 rpy=0 0 0, axis 0 0 0

Commit message: update

File: urdf/hephaestus_description.urdf (robot description, URDF)
Before this commit: robot hephaestus_description, 8 links, 7 joints
Joints:
- joint j1: axis 0 0 1 -> 0 0 -1; limit lower=-3.141592653589793116 upper=3.141592653589793116 effort=1 velocity=20 -> lower=-3.141592653589793116 upper=3.141592653589793116 effort=1 velocity=0.7
- joint j2: axis 0 0 1 -> 0 0 -1; limit lower=-3.141592653589793116 upper=3.141592653589793116 effort=1 velocity=20 -> lower=-3.141592653589793116 upper=3.141592653589793116 effort=1 velocity=0.7
- joint j3: limit lower=-3.141592653589793116 upper=3.141592653589793116 effort=1 velocity=20 -> lower=-3.141592653589793116 upper=3.141592653589793116 effort=1 velocity=0.7
- joint j4: limit lower=-3.141592653589793116 upper=3.141592653589793116 effort=1 velocity=20 -> lower=-3.141592653589793116 upper=3.141592653589793116 effort=1 velocity=0.7
- joint j5: limit lower=-3.141592653589793116 upper=3.141592653589793116 effort=1 velocity=20 -> lower=-3.141592653589793116 upper=3.141592653589793116 effort=1 velocity=0.7
- joint j6: limit lower=-3.141592653589793116 upper=3.141592653589793116 effort=1 velocity=20 -> lower=-3.141592653589793116 upper=3.141592653589793116 effort=1 velocity=0.7

Commit message: corl edit

File: urdf/hephaestus_description.urdf (robot description, URDF)
Before this commit: robot hephaestus_description, 8 links, 7 joints
Links:
- link gripper: geometry collision mesh filename=package://hephaestus_description/meshes/4005_convertor.stl; collision mesh filename=package://hephaestus_description/meshes/4036_out_type_b.stl

Commit message: update

File: urdf/hephaestus_description.urdf (robot description, URDF)
Before this commit: robot hephaestus_description, 8 links, 7 joints
Links:
- added link world
Joints:
- added joint fix_to_World: type fixed, parent world, child link1, origin xyz=0 0 0 rpy=0 0 0, axis 0 0 0
- joint j1: limit lower=-3.141592653589793116 upper=3.141592653589793116 effort=1 velocity=0.7 -> lower=-3.141592653589793116 upper=3.141592653589793116 effort=50 velocity=6.28
- joint j2: limit lower=-3.141592653589793116 upper=3.141592653589793116 effort=1 velocity=0.7 -> lower=-3.141592653589793116 upper=3.141592653589793116 effort=50 velocity=6.28
- joint j3: limit lower=-3.141592653589793116 upper=3.141592653589793116 effort=1 velocity=0.7 -> lower=-3.141592653589793116 upper=3.141592653589793116 effort=50 velocity=6.28
- joint j4: limit lower=-3.141592653589793116 upper=3.141592653589793116 effort=1 velocity=0.7 -> lower=-3.141592653589793116 upper=3.141592653589793116 effort=50 velocity=6.28
- joint j5: limit lower=-3.141592653589793116 upper=3.141592653589793116 effort=1 velocity=0.7 -> lower=-3.141592653589793116 upper=3.141592653589793116 effort=50 velocity=6.28
- joint j6: limit lower=-3.141592653589793116 upper=3.141592653589793116 effort=1 velocity=0.7 -> lower=-3.141592653589793116 upper=3.141592653589793116 effort=50 velocity=6.28
